File: Vectr_Board_Files/Vectr_1_3.brd (EAGLE design)
At the start: 50 x 107 mm, 110 parts, among them IC1 TL074D, U1 MCP3201-CI/SN, U2 DAC8554, U3 MCP1755S, U4 MCP1755S, U5 LM4040, U6 23LC512, U7 SST25VF010A, U8 PIC32MX430-QFP

Commit message: Interim Board Update
Parts:
- removed F1, F2: PTCSMD, SparkFun-PowerIC:PTC-1206
- removed R29: 10k, SparkFun-Passives:0402-RES
- added D2, D3: MBR0520LT, diode:SOD123
- C15: value 4.7uF -> 47uF
- R28: value 10k -> 1.8k
- moved R28 0.75 mm to (37.4, 75.5)
Connections:
- net ANALOG_REFERENCE: no longer R29.1
- net N$42: now also D2.A; no longer F1.1
- net N$44: now also D3.C; no longer F2.1
- net VCC: now also D2.C; no longer F1.2, R29.2
- net VEE: now also D3.A; no longer F2.2
Routing:
- net VCC: track 112.3 -> 110.8 mm
- net ANALOG_REFERENCE: track 31.8 -> 30.7 mm
- net VEE: track 20.0 -> 19.0 mm
Other:
- board text added: "The connector is at 30.5 and 44.25 with the position being between the top two positions."

Commit message: Changing connectors
Parts:
- removed TO_SENSOR: M50-3101045, HackMe:M50-3101045
- added U$1: EURO_POWER_TH, HackMe:EURO_POWER_TH
- POWER: value 16-SMT -> EURO_POWER_TH; device HackMe:16-SMT -> HackMe:EURO_POWER_TH
- moved U1 3.01 mm to (33.5, 59.1)
Connections:
- net 5V: now also U$1.1; no longer TO_SENSOR.1, TO_SENSOR.20
- net AGND: no longer TO_SENSOR.11
- net GND: now also POWER.10, POWER.11, POWER.12, POWER.13, POWER.14, POWER.9; no longer POWER.P$10, POWER.P$11, POWER.P$12, POWER.P$13, POWER.P$14, POWER.P$9, TO_SENSOR.10
- net I2C1_SCL: now also U$1.3; no longer TO_SENSOR.2
- net I2C1_SDA: no longer TO_SENSOR.19
- net LED_PWM_1: now also U$1.9; no longer TO_SENSOR.5
- net LED_PWM_2: no longer TO_SENSOR.16
- net LED_PWM_3: now also U$1.11; no longer TO_SENSOR.6
- net LED_PWM_4: no longer TO_SENSOR.15
- net LED_PWM_5: now also U$1.13; no longer TO_SENSOR.7
- net MGC3130_IRQ: no longer TO_SENSOR.18
- net MGC3130_RESET: now also U$1.5; no longer TO_SENSOR.3
- net N$42: now also POWER.7, POWER.8; no longer POWER.P$7, POWER.P$8
- net N$44: now also POWER.15, POWER.16; no longer POWER.P$15, POWER.P$16
- net SR_CLK: no longer TO_SENSOR.17
- net SR_DATA: now also U$1.7; no longer TO_SENSOR.4
Routing:
- net GND: track 193.6 -> 199.1 mm
- net 5V: track 65.1 -> 59.7 mm
- net ANALOG_REFERENCE: track 30.7 -> 35.8 mm
- net N$44: track 29.2 -> 32.9 mm
- net SPI1_CLK: track 45.5 -> 48.5 mm
- net SPI1_MISO: track 37.7 -> 40.7 mm
- net ADC_SPI_EN: track 49.5 -> 52.5 mm
- net N$24: track 40.9 -> 42.7 mm
- net AGND: track 109.0 -> 110.4 mm
- net LED_PWM_2: track 17.3 -> 16.0 mm
- net SR_CLK: track 28.2 -> 26.9 mm
- net LED_PWM_4: track 9.56 -> 8.40 mm

Commit message: Preliminary Final Revision
Parts:
- removed ICSP: PIC-ICSPPTH, SparkFun-Connectors:MOLEX-1X6
- added J1: (no value), tag-connect:TC2030-MCP
- EXP1, EXP2: device SparkFun-Connectors:1X04_SMD_STRAIGHT_COMBO -> SparkFun-Connectors:1X04
- moved D3 107.2 mm to (48.5, 88.5), turned to 90 degrees
- moved D2 100.8 mm to (45.5, 88.5), turned to 270 degrees
- moved EXP2 17.5 mm to (48.6, 43.3)
- moved C13 17.1 mm to (46.2, 51.9), turned to 270 degrees
- moved U4 13.9 mm to (46.3, 57.7)
- moved C12 13.9 mm to (43.7, 51.8), turned to 90 degrees
- moved EXP1 7.27 mm to (45.1, 30.9)
- moved C23 5.54 mm to (31.8, 33.5)
- moved POWER 4.50 mm to (47.0, 84.0)
- moved R6 4.26 mm to (41.7, 57.7)
- moved D1 4.00 mm to (38.5, 55.5)
- moved C1 3.34 mm to (34.0, 56.0)
- moved C24 1.46 mm to (33.1, 33.5)
- moved R19 1.00 mm to (42.3, 87.0)
- moved R3 0.82 mm to (40.8, 65.8)
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- renumbered U$1 to TO_SENSOR
Connections:
- net 3.3V: now also J1.2; no longer ICSP.5
- net 5V: now also TO_SENSOR.2
- net AGND: now also TO_SENSOR.16
- net GND: now also J1.3, TO_SENSOR.15; no longer ICSP.4
- net I2C1_SDA: now also TO_SENSOR.4
- net LED_PWM_2: now also TO_SENSOR.10
- net LED_PWM_4: now also TO_SENSOR.12
- net MCLR: now also J1.1; no longer ICSP.6
- net MGC3130_IRQ: now also TO_SENSOR.6
- net PGEC: now also J1.5; no longer ICSP.2
- net PGED: now also J1.4; no longer ICSP.3
- net SR_CLK: now also TO_SENSOR.8
Routing:
- net GND: track 199.1 -> 148.1 mm, vias 31 -> 24
- net VCC: track 110.8 -> 72.8 mm, vias 2 -> 0
- net 5V: track 59.7 -> 92.2 mm, vias 8 -> 6
- net I2C2_SCL: track 50.8 -> 34.3 mm, vias 3 -> 1
- net 3.3V: track 194.4 -> 181.2 mm, vias 18 -> 14
- net LED_PWM_2: track 16.0 -> 27.3 mm
- net SPI1_CLK: track 48.5 -> 37.7 mm, vias 3 -> 2
- net I2C2_SDA: track 48.5 -> 38.3 mm
- net MCLR: track 22.1 -> 31.6 mm, vias 1 -> 2
- net LED_PWM_5: track 19.8 -> 10.4 mm, vias 2 -> 0
- net LDAC: track 48.1 -> 56.8 mm
- net I2C1_SCL: track 40.6 -> 33.1 mm
- net LED_PWM_4: track 8.40 -> 15.5 mm
- net SR_CLK: track 26.9 -> 33.6 mm
- net PGEC: track 20.1 -> 26.6 mm, vias 0 -> 1
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