File: Vectr_Board_Files/Vectr_1_3.sch (EAGLE design)
At the start: 108 parts, among them IC1 TL074D, U1 MCP3201-CI/SN, U2 DAC8554, U3 MCP1755S, U4 MCP1755S, U5 LM4040, U6 23LC512, U7 SST25VF010A, U8 PIC32MX430-QFP

Commit message: Interim Board Update
Parts:
- removed F1, F2: PTCSMD, SparkFun-PowerIC:PTCSMD
- removed R29: 10k, SparkFun-Passives:RESISTOR0402-RES
- added D2, D3: MBR0520LT, diode:MBR0520LT
- C15: value 4.7uF -> 47uF
- R28: value 10k -> 1.8k
Connections:
- net ANALOG_REFERENCE: no longer R29.1
- net N$42: now also D2.A; no longer F1.1
- net N$44: now also D3.C; no longer F2.1
- net VCC: now also D2.C; no longer F1.2, R29.2
- net VEE: now also D3.A; no longer F2.2
Other:
- moved on the sheet: R28
Changed lines of the file:
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@@
 <part name="FRAME3" library="frames" deviceset="FRAME_A_L" device=""/>
 <part name="U4" library="HackMe" deviceset="MCP1755S" device=""/>
-<part name="F1" library="SparkFun-PowerIC" deviceset="PTC" device="SMD"/>
-<part name="F2" library="SparkFun-PowerIC" deviceset="PTC" device="SMD"/>
 <part name="P+4" library="supply1" deviceset="VCC" device=""/>
 <part name="SUPPLY14" library="supply2" deviceset="VEE" device=""/>
@@
 <part name="SUPPLY9" library="SparkFun-Aesthetics" deviceset="3.3V" device=""/>
 <part name="SUPPLY29" library="SparkFun-Aesthetics" deviceset="3.3V" device=""/>
-<part name="C15" library="SparkFun-Capacitors" deviceset="CAP" device="0805" value="4.7uF"/>
+<part name="C15" library="SparkFun-Capacitors" deviceset="CAP" device="0805" value="47uF"/>
 <part name="C14" library="SparkFun-Passives" deviceset="CAP" device="0805" value="4.7uF"/>
 <part name="R27" library="SparkFun-Passives" deviceset="RESISTOR" device="0402-RES" value="1k"/>
@@
 <part name="SUPPLY10" library="SparkFun-Aesthetics" deviceset="5V" device=""/>
 <part name="U5" library="HackMe" deviceset="LM4040" device=""/>
-<part name="R29" library="SparkFun-Passives" deviceset="RESISTOR" device="0402-RES" value="10k"/>
-<part name="R28" library="SparkFun-Passives" deviceset="RESISTOR" device="0402-RES" value="10k"/>
+<part name="R28" library="SparkFun-Passives" deviceset="RESISTOR" device="0402-RES" value="1.8k"/>
 <part name="C1" library="SparkFun-Passives" deviceset="CAP" device="0402-CAP" value=".1uF"/>
 <part name="AGND15" library="supply1" deviceset="AGND" device=""/>
@@
 <part name="R41" library="SparkFun-Passives" deviceset="RESISTOR" device="0402-RES" value="10k"/>
 <part name="R42" library="SparkFun-Passives" deviceset="RESISTOR" device="0402-RES" value="33"/>
+<part name="D2" library="diode" deviceset="MBR0520LT" device=""/>
+<part name="D3" library="diode" deviceset="MBR0520LT" device=""/>
 </parts>
 <sheets>
@@
 <instance part="FRAME3" gate="G$2" x="172.72" y="0"/>
 <instance part="U4" gate="G$1" x="121.92" y="127"/>
-<instance part="F1" gate="G$1" x="114.3" y="193.04"/>
-<instance part="F2" gate="G$1" x="114.3" y="177.8"/>
 <instance part="P+4" gate="VCC" x="147.32" y="203.2"/>
 <instance part="SUPPLY14" gate="G$1" x="147.32" y="170.18" rot="R180"/>
@@
 <instance part="POWER" gate="G$1" x="76.2" y="187.96"/>
 <instance part="P+1" gate="VCC" x="30.48" y="139.7"/>
-<instance part="P+2" gate="VCC" x="177.8" y="142.24"/>
+<instance part="P+2" gate="VCC" x="177.8" y="134.62"/>
 <instance part="TO_SENSOR" gate="G$1" x="187.96" y="180.34"/>
 <instance part="U3" gate="G$1" x="58.42" y="127"/>
 <instance part="P+5" gate="VCC" x="109.22" y="137.16"/>
 <instance part="U5" gate="G$1" x="195.58" y="124.46" rot="R90"/>
-<instance part="R29" gate="G$1" x="185.42" y="129.54" rot="R180"/>
-<instance part="R28" gate="G$1" x="185.42" y="137.16" rot="R180"/>
+<instance part="R28" gate="G$1" x="185.42" y="129.54" rot="R180"/>
+<instance part="D2" gate="G$1" x="114.3" y="193.04"/>
+<instance part="D3" gate="G$1" x="116.84" y="177.8" rot="R180"/>
 </instances>
 <busses>
@@
 <wire x1="91.44" y1="187.96" x2="99.06" y2="187.96" width="0.1524" layer="91"/>
 <wire x1="99.06" y1="187.96" x2="99.06" y2="193.04" width="0.1524" layer="91"/>
-<pinref part="F1" gate="G$1" pin="1"/>
-<wire x1="99.06" y1="193.04" x2="109.22" y2="193.04" width="0.1524" layer="91"/>
+<wire x1="99.06" y1="193.04" x2="111.76" y2="193.04" width="0.1524" layer="91"/>
 <wire x1="99.06" y1="193.04" x2="99.06" y2="203.2" width="0.1524" layer="91"/>
 <junction x="99.06" y="193.04"/>
@@
 <pinref part="POWER" gate="G$1" pin="7"/>
 <pinref part="POWER" gate="G$1" pin="8"/>
+<pinref part="D2" gate="G$1" pin="A"/>
 </segment>
 </net>
 <net name="N$44" class="0">
 <segment>
-<pinref part="F2" gate="G$1" pin="1"/>
 <wire x1="91.44" y1="177.8" x2="99.06" y2="177.8" width="0.1524" layer="91"/>
-<wire x1="99.06" y1="177.8" x2="109.22" y2="177.8" width="0.1524" layer="91"/>
+<wire x1="99.06" y1="177.8" x2="114.3" y2="177.8" width="0.1524" layer="91"/>
 <wire x1="99.06" y1="177.8" x2="99.06" y2="165.1" width="0.1524" layer="91"/>
 <junction x="99.06" y="177.8"/>
@@
 <pinref part="POWER" gate="G$1" pin="15"/>
 <pinref part="POWER" gate="G$1" pin="16"/>
+<pinref part="D3" gate="G$1" pin="C"/>
 </segment>
 </net>
@@
 <pinref part="SUPPLY14" gate="G$1" pin="VEE"/>
 <wire x1="147.32" y1="177.8" x2="147.32" y2="172.72" width="0.1524" layer="91"/>
-<pinref part="F2" gate="G$1" pin="2"/>
-<wire x1="121.92" y1="177.8" x2="147.32" y2="177.8" width="0.1524" layer="91"/>
+<wire x1="119.38" y1="177.8" x2="147.32" y2="177.8" width="0.1524" layer="91"/>
+<pinref part="D3" gate="G$1" pin="A"/>
 </segment>
 </net>
@@
 <pinref part="P+4" gate="VCC" pin="VCC"/>
 <wire x1="147.32" y1="198.12" x2="147.32" y2="200.66" width="0.1524" layer="91"/>
-<pinref part="F1" gate="G$1" pin="2"/>
-<wire x1="121.92" y1="193.04" x2="129.54" y2="193.04" width="0.1524" layer="91"/>
+<wire x1="116.84" y1="193.04" x2="129.54" y2="193.04" width="0.1524" layer="91"/>
 <wire x1="129.54" y1="193.04" x2="129.54" y2="198.12" width="0.1524" layer="91"/>
 <wire x1="129.54" y1="198.12" x2="147.32" y2="198.12" width="0.1524" layer="91"/>
+<pinref part="D2" gate="G$1" pin="C"/>
 </segment>
 <segment>
@@
 <pinref part="C14" gate="G$1" pin="2"/>
 <pinref part="P+2" gate="VCC" pin="VCC"/>
-<wire x1="177.8" y1="139.7" x2="177.8" y2="137.16" width="0.1524" layer="91"/>
-<pinref part="R29" gate="G$1" pin="2"/>
-<wire x1="177.8" y1="137.16" x2="177.8" y2="129.54" width="0.1524" layer="91"/>
+<wire x1="177.8" y1="132.08" x2="177.8" y2="129.54" width="0.1524" layer="91"/>
 <wire x1="177.8" y1="129.54" x2="177.8" y2="127" width="0.1524" layer="91"/>
-<wire x1="180.34" y1="129.54" x2="177.8" y2="129.54" width="0.1524" layer="91"/>
+<pinref part="R28" gate="G$1" pin="2"/>
+<wire x1="177.8" y1="129.54" x2="180.34" y2="129.54" width="0.1524" layer="91"/>
 <junction x="177.8" y="129.54"/>
-<pinref part="R28" gate="G$1" pin="2"/>
-<wire x1="177.8" y1="137.16" x2="180.34" y2="137.16" width="0.1524" layer="91"/>
-<junction x="177.8" y="137.16"/>
 </segment>
 <segment>
@@
 <wire x1="210.82" y1="124.46" x2="210.82" y2="129.54" width="0.1524" layer="91"/>
 <label x="210.82" y="129.54" size="1.778" layer="95"/>
-<pinref part="R29" gate="G$1" pin="1"/>
 <pinref part="U5" gate="G$1" pin="C"/>
-<wire x1="190.5" y1="129.54" x2="193.04" y2="129.54" width="0.1524" layer="91"/>
-<wire x1="193.04" y1="129.54" x2="195.58" y2="129.54" width="0.1524" layer="91"/>
 <wire x1="195.58" y1="129.54" x2="195.58" y2="127" width="0.1524" layer="91"/>
 <junction x="195.58" y="129.54"/>
 <pinref part="R28" gate="G$1" pin="1"/>
-<wire x1="190.5" y1="137.16" x2="193.04" y2="137.16" width="0.1524" layer="91"/>
-<wire x1="193.04" y1="137.16" x2="193.04" y2="129.54" width="0.1524" layer="91"/>
-<junction x="193.04" y="129.54"/>
-</segment>
-</net>
+<wire x1="190.5" y1="129.54" x2="195.58" y2="129.54" width="0.1524" layer="91"/>
+</segment>
+</net>

Commit message: Preliminary Final Revision
Parts:
- removed ICSP: PIC-ICSPPTH, SparkFun-Connectors:PIC-ICSPPTH
- added J1: (no value), tag-connect:TC2030-MCP
- EXP1, EXP2: device SparkFun-Connectors:M04SMD_STRAIGHT_COMBO -> SparkFun-Connectors:M04PTH
- POWER: value 16-SMT -> EURO_POWER_TH; device HackMe:16-SMT -> HackMe:EURO_POWER_TH
- TO_SENSOR: value M50-3101045 -> EURO_POWER_TH; device HackMe:M50-3101045 -> HackMe:EURO_POWER_TH
Connections:
- net 3.3V: now also J1.VDD; no longer ICSP.VCC
- net 5V: now also TO_SENSOR.2; no longer TO_SENSOR.20
- net AGND: now also TO_SENSOR.16; no longer TO_SENSOR.11
- net GND: now also J1.VSS(GND), TO_SENSOR.15; no longer ICSP.GND, TO_SENSOR.10
- net I2C1_SCL: now also TO_SENSOR.3; no longer TO_SENSOR.2
- net I2C1_SDA: now also TO_SENSOR.4; no longer TO_SENSOR.19
- net LED_PWM_1: now also TO_SENSOR.9; no longer TO_SENSOR.5
- net LED_PWM_2: now also TO_SENSOR.10; no longer TO_SENSOR.16
- net LED_PWM_3: now also TO_SENSOR.11; no longer TO_SENSOR.6
- net LED_PWM_4: now also TO_SENSOR.12; no longer TO_SENSOR.15
- net LED_PWM_5: now also TO_SENSOR.13; no longer TO_SENSOR.7
- net MCLR: now also J1.VPP/MCLR; no longer ICSP.VPP
- net MGC3130_IRQ: now also TO_SENSOR.6; no longer TO_SENSOR.18
- net MGC3130_RESET: now also TO_SENSOR.5; no longer TO_SENSOR.3
- net PGEC: now also J1.ICSP_CLK/PGC; no longer ICSP.PGC
- net PGED: now also J1.ICSP_DAT/PGD; no longer ICSP.PGD
- net SR_CLK: now also TO_SENSOR.8; no longer TO_SENSOR.17
- net SR_DATA: now also TO_SENSOR.7; no longer TO_SENSOR.4
